Commit message: Imported upstream version '0.5.0' of 'upstream'

File: kobuki_description/urdf/kobuki_gazebo.urdf.xacro (robot description, xacro)
@@ -32,5 +32,5 @@
 	      <visualize>true</visualize>
 	      <contact>
-	        <collision>base_footprint_geom_base_link</collision>
+	        <collision>base_footprint_collision_base_link</collision>
 	      </contact>
 	    </sensor>
@@ -120,19 +120,31 @@
 	    </sensor>
 	  </gazebo>
-	  <gazebo>
-	    <plugin name="imu_controller" filename="libgazebo_ros_imu.so">
-	      <alwaysOn>true</alwaysOn>
-	      <updateRate>50</updateRate>
-	      <bodyName>gyro_link</bodyName>
-	      <topicName>/mobile_base/sensors/imu_data</topicName>
-	      <serviceName>imu/is_calibrated</serviceName>
-	      <gaussianNoise>${0.0017*0.0017}</gaussianNoise>
-	      <xyzOffsets>0 0 0</xyzOffsets>
-	      <rpyOffsets>0 0 0</rpyOffsets>
-	    </plugin>
+	  <gazebo reference="gyro_link">
+	   <sensor type="imu" name="imu">
+        <always_on>true</always_on>
+        <update_rate>50</update_rate>
+        <visualize>false</visualize>
+        <imu>
+          <noise>
+            <type>gaussian</type>
+	          <rate>
+	            <mean>0.0</mean>
+	            <stddev>${0.0014*0.0014}</stddev> <!-- 0.25 x 0.25 (deg/s) -->
+	            <bias_mean>0.0</bias_mean>
+	            <bias_stddev>0.0</bias_stddev>
+	          </rate>
+		        <accel> <!-- not used in the plugin and real robot, hence using tutorial values -->
+			        <mean>0.0</mean>
+			        <stddev>1.7e-2</stddev>
+			        <bias_mean>0.1</bias_mean>
+			        <bias_stddev>0.001</bias_stddev>
+		        </accel>
+          </noise>
+	      </imu>
+      </sensor>
 	  </gazebo>
 	  <gazebo>
 	    <plugin name="kobuki_controller" filename="libgazebo_ros_kobuki.so">
-	      <publish_tf>0</publish_tf>
+	      <publish_tf>1</publish_tf>
 	      <left_wheel_joint_name>wheel_left_joint</left_wheel_joint_name>
 	      <right_wheel_joint_name>wheel_right_joint</right_wheel_joint_name>
@@ -142,9 +154,9 @@
 	      <velocity_command_timeout>0.6</velocity_command_timeout>
 	      <cliff_sensor_left_name>cliff_sensor_left</cliff_sensor_left_name>
-	      <cliff_sensor_front_name>cliff_sensor_front</cliff_sensor_front_name>
+	      <cliff_sensor_center_name>cliff_sensor_front</cliff_sensor_center_name>
 	      <cliff_sensor_right_name>cliff_sensor_right</cliff_sensor_right_name>
 	      <cliff_detection_threshold>0.04</cliff_detection_threshold>
 	      <bumper_name>bumpers</bumper_name>
-	      <base_collision_model_link>base_link</base_collision_model_link>
+        <imu_name>imu</imu_name>
 	    </plugin>
 	  </gazebo>
