Commit message: Imported upstream version '0.4.0' of 'upstream'

File: kobuki_description/urdf/kobuki.urdf.xacro (robot description, xacro)
@@ -7,26 +7,9 @@
  -->
 <robot name="kobuki" xmlns:xacro="http://ros.org/wiki/xacro">
-  <include filename="$(find kobuki_description)/urdf/common_properties.urdf.xacro"/>
-  <include filename="$(find kobuki_description)/urdf/kobuki_gazebo.urdf.xacro"/>
-  <!-- Xacro properties -->
-  <xacro:property name="M_SCALE" value="0.001"/>
+  <xacro:include filename="$(find kobuki_description)/urdf/common_properties.urdf.xacro"/>
   <!-- Kobuki -->
   <xacro:macro name="kobuki">
-    <link name="base_footprint">
-      <visual>
-        <origin xyz="0 0 0" rpy="0 0 0"/>
-        <geometry>
-          <box size="0.001 0.001 0.001"/>
-        </geometry>
-        <xacro:insert_block name="material_black" />
-      </visual>
-      <collision>
-        <origin xyz="0 0 0.035" rpy="0 0 0"/>
-        <geometry>
-         <box size="0.001 0.001 0.001"/>
-        </geometry>
-      </collision>
-    </link>
-     <!--
+    <link name="base_footprint"/>
+    <!--
        Base link is set at the bottom of the base mould.
        This is done to be compatible with the way base link
@@ -45,25 +28,29 @@
       <visual>
         <geometry>
-          <mesh filename="package://kobuki_description/meshes/base.dae" scale="${M_SCALE} ${M_SCALE} ${M_SCALE}"/>
-        </geometry>
-        <origin xyz="0.0 0 0.05469" rpy="${M_PI/2} 0 ${M_PI/2}"/>
-        <xacro:insert_block name="material_black"/>
+          <!-- new mesh -->
+          <mesh filename="package://kobuki_description/meshes/main_body.dae" />
+        </geometry>
+        <origin xyz="0.001 0 0.05199" rpy="0 0 0"/>
       </visual>
       <collision>
         <geometry>
-          <cylinder length="0.10938" radius="0.175615"/>
-        </geometry>
-        <origin xyz="0.0 0.0 0.05469" rpy="0 0 0"/>
-      </collision>
-      <inertial>
+          <cylinder length="0.10938" radius="0.176"/>
+        </geometry>
+        <origin xyz="0.0 0 0.05949" rpy="0 0 0"/>
+      </collision>
+      <inertial>
+        <origin xyz="0 0 0"/>
         <mass value="2.4"/> <!-- 2.4/2.6 kg for small/big battery pack -->
-        <origin xyz="0 0 0"/>
-        <inertia ixx="0.0001" ixy="0.0" ixz="0.0"
-                 iyy="0.0001" iyz="0.0"
-                 izz="0.0001" />
-      </inertial>
-      <gazebo reference="base_link">
-        <material>Gazebo/Black</material>
-      </gazebo>
+        <!-- http://en.wikipedia.org/wiki/List_of_moment_of_inertia_tensors
+             Assuming homogeneous mass distribution
+		         m=2.4; h=0.09; r=0.175;
+		         ixx = 1/12*m*(3*r^2 + h^2)
+		         iyy = 1/12*m*(3*r^2 + h^2)
+		         izz = 1/2*m*r^2
+          -->
+        <inertia ixx="0.019995" ixy="0.0" ixz="0.0"
+                 iyy="0.019995" iyz="0.0"
+                 izz="0.006125" />
+      </inertial>
     </link>
     <joint name="wheel_left_joint" type="continuous">
@@ -76,8 +63,7 @@
       <visual>
         <geometry>
-          <mesh filename="package://kobuki_description/meshes/wheel.dae" scale="${M_SCALE} ${M_SCALE} ${M_SCALE}"/>
-        </geometry>
-        <origin xyz="0 0 0" rpy="0 ${M_PI/2} 0"/>
-        <xacro:insert_block name="material_black"/>
+          <mesh filename="package://kobuki_description/meshes/wheel.dae"/>
+        </geometry>
+        <origin xyz="0 0 0" rpy="0 0 0"/>
       </visual>
       <collision>
@@ -104,8 +90,7 @@
       <visual>
         <geometry>
-          <mesh filename="package://kobuki_description/meshes/wheel.dae" scale="${M_SCALE} ${M_SCALE} ${M_SCALE}"/>
-        </geometry>
-        <origin xyz="0 0 0" rpy="0 ${M_PI/2} 0"/>
-        <xacro:insert_block name="material_black"/>
+          <mesh filename="package://kobuki_description/meshes/wheel.dae"/>
+        </geometry>
+        <origin xyz="0 0 0" rpy="0 0 0"/>
       </visual>
       <collision>
@@ -123,9 +108,48 @@
       </inertial>
     </link>
+    <joint name="caster_front_joint" type="fixed">
+      <parent link="base_link"/>
+      <child link="caster_front_link"/>
+      <origin xyz="0.115 0.0 0.007" rpy="${-M_PI/2} 0 0"/>
+    </joint>
+    <link name="caster_front_link">
+      <collision>
+        <geometry>
+          <cylinder length="0.0176" radius="0.017"/>
+        </geometry>
+        <origin rpy="0 0 0" xyz="0 0 0"/>
+      </collision>
+      <inertial>
+        <mass value="0.01" />
+        <origin xyz="0 0 0" />
+        <inertia ixx="0.001" ixy="0.0" ixz="0.0"
+                 iyy="0.001" iyz="0.0"
+                 izz="0.001" />
+      </inertial>
+    </link>
+    <joint name="caster_back_joint" type="fixed">
+      <parent link="base_link"/>
+      <child link="caster_back_link"/>
+      <origin xyz="-0.135 0.0 0.009" rpy="${-M_PI/2} 0 0"/>
+    </joint>
+    <link name="caster_back_link">
+      <collision>
+        <geometry>
+          <cylinder length="0.0176" radius="0.017"/>
+        </geometry>
+        <origin rpy="0 0 0" xyz="0 0 0"/>
+      </collision>
+      <inertial>
+        <mass value="0.01" />
+        <origin xyz="0 0 0" />
+        <inertia ixx="0.001" ixy="0.0" ixz="0.0"
+                 iyy="0.001" iyz="0.0"
+                 izz="0.001" />
+      </inertial>
+    </link>
     <!-- Kobuki's sensors -->
-    <!-- TODO: Check placement! -->
     <joint name="gyro_joint" type="fixed">
       <axis xyz="0 1 0"/>
-      <origin xyz="0 0 0.058" rpy="0 0 0"/>
+      <origin xyz="0.056 0.062 0.0202" rpy="0 0 0"/>
       <parent link="base_link"/>
       <child link="gyro_link"/>
@@ -140,10 +164,10 @@
       </inertial>
     </link>
-	  <joint name="cliff_sensor_left_joint" type="fixed">
-	    <origin xyz="0.07 0.14 0.028" rpy="0 ${M_PI/2} 0" />
-	    <parent link="base_link"/>
-	    <child link="cliff_sensor_left_link" />
-	  </joint>
-	  <link name="cliff_sensor_left_link">
+    <joint name="cliff_sensor_left_joint" type="fixed">
+      <origin xyz="0.08734 0.13601 0.0214" rpy="0 ${M_PI/2} 0" />
+      <parent link="base_link"/>
+      <child link="cliff_sensor_left_link" />
+    </joint>
+    <link name="cliff_sensor_left_link">
       <inertial>
         <mass value="0.0001" />
@@ -154,9 +178,9 @@
       </inertial>
     </link>
-	  <joint name="cliff_sensor_right_joint" type="fixed">
-	    <origin xyz="0.07 -0.14 0.028" rpy="0 ${M_PI/2} 0" />
-	    <parent link="base_link"/>
-	    <child link="cliff_sensor_right_link" />
-	  </joint>
+    <joint name="cliff_sensor_right_joint" type="fixed">
+      <origin xyz="0.085 -0.13601 0.0214" rpy="0 ${M_PI/2} 0" />
+      <parent link="base_link"/>
+      <child link="cliff_sensor_right_link" />
+    </joint>
     <link name="cliff_sensor_right_link">
       <inertial>
@@ -169,5 +193,5 @@
     </link>
     <joint name="cliff_sensor_front_joint" type="fixed">
-      <origin xyz="0.18 0.00 0.028" rpy="0 ${M_PI/2} 0" />
+      <origin xyz="0.156 0.00 0.0214" rpy="0 ${M_PI/2} 0" />
       <parent link="base_link"/>
       <child link="cliff_sensor_front_link" />
@@ -182,8 +206,4 @@
       </inertial>
     </link>
-    <!--  Gazebo additions -->
-    <kobuki_sim/>
-    <kobuki_cliff_sensors/>
-    <turtlebot_sim_imu/>
   </xacro:macro>
 </robot>

File: kobuki_description/urdf/kobuki_gazebo.urdf.xacro (robot description, xacro)
@@ -1,103 +1,148 @@
 <?xml version="1.0"?>
-<robot xmlns:controller="http://playerstage.sourceforge.net/gazebo/xmlschema/#controller"
-       xmlns:interface="http://playerstage.sourceforge.net/gazebo/xmlschema/#interface"
-       xmlns:sensor="http://playerstage.sourceforge.net/gazebo/xmlschema/#sensor"
-       xmlns:xacro="http://ros.org/wiki/xacro"
-       name="turtlebot_gazebo">
-<xacro:macro name="kobuki_sim">
-  <gazebo>
-    <controller:gazebo_ros_kobuki name="kobuki_controller" plugin="libgazebo_ros_kobuki.so">
-      <alwaysOn>true</alwaysOn>
-      <node_namespace>kobuki_node</node_namespace>
-      <left_wheel_joint>wheel_left_joint</left_wheel_joint>
-      <right_wheel_joint>wheel_right_joint</right_wheel_joint>
-      <wheel_separation>.230</wheel_separation>
-      <wheel_diameter>0.070</wheel_diameter>
-      <base_geom>base_footprint</base_geom>
-      <updateRate>40</updateRate>
-      <torque>1.0</torque>
-    </controller:gazebo_ros_kobuki>
-  </gazebo>
+<robot>
   <gazebo reference="wheel_left_link">
-    <mu1 value="10"/>
-    <mu2 value="10"/>
-    <kp value="100000000.0"/>
-    <kd value="10000.0"/>
-    <fdir value="1 0 0"/>
+    <mu1>1.0</mu1>
+    <mu2>1.0</mu2>
+    <kp>100000000.0</kp>
+    <kd>10000.0</kd>
   </gazebo>
   <gazebo reference="wheel_right_link">
-    <mu1 value="10"/>
-    <mu2 value="10"/>
-    <kp value="100000000.0"/>
-    <kd value="10000.0"/>
-    <fdir value="1 0 0"/>
+    <mu1>1.0</mu1>
+    <mu2>1.0</mu2>
+    <kp>100000000.0</kp>
+    <kd>10000.0</kd>
   </gazebo>
   <gazebo reference="caster_front_link">
-    <mu1 value="0"/>
-    <mu2 value="0"/>
-    <kp value="100000000.0"/>
-    <kd value="10000.0"/>
+    <mu1>0.0</mu1>
+    <mu2>0.0</mu2>
+    <kp>100000000.0</kp>
+    <kd>10000.0</kd>
   </gazebo>
   <gazebo reference="caster_back_link">
-    <mu1 value="0"/>
-    <mu2 value="0"/>
-    <kp value="100000000.0"/>
-    <kd value="10000.0"/>
+    <mu1>0.0</mu1>
+    <mu2>0.0</mu2>
+    <kp>100000000.0</kp>
+    <kd>10000.0</kd>
   </gazebo>
-</xacro:macro>
-<xacro:macro name="kobuki_cliff_sensors">
+  <gazebo reference="base_link">
+    <sensor type="contact" name="bumpers">
+      <always_on>1</always_on>
+      <update_rate>50.0</update_rate>
+      <visualize>true</visualize>
+      <contact>
+        <collision>base_footprint_geom_base_link</collision>
+      </contact>
+    </sensor>
+  </gazebo>
   <gazebo reference="cliff_sensor_left_link">
-    <sensor:ray name="cliff_sensor_left">
-      <alwaysActive>true</alwaysActive>
-      <rayCount>1</rayCount>
-      <rangeCount>1</rangeCount>
-      <resRange>0.1</resRange>
-      <minAngle>0</minAngle>
-      <maxAngle>0</maxAngle>
-      <minRange>0.01</minRange>
-      <maxRange>0.04</maxRange>
-      <displayRays>false</displayRays>
-    </sensor:ray>
+    <sensor type="ray" name="cliff_sensor_left">
+      <always_on>true</always_on>
+      <update_rate>50</update_rate>
+      <visualize>true</visualize>
+      <ray>
+        <scan>
+          <horizontal>
+            <samples>50</samples>
+            <resolution>1.0</resolution>
+            <min_angle>-0.0436</min_angle>  <!-- -2.5 degree -->
+            <max_angle>0.0436</max_angle> <!-- 2.5 degree -->
+          </horizontal>
+          <vertical>
+            <samples>50</samples>
+            <resolution>1.0</resolution>
+            <min_angle>-0.0436</min_angle>  <!-- -2.5 degree -->
+            <max_angle>0.0436</max_angle> <!-- 2.5 degree -->
+          </vertical>
+        </scan>
+        <range>
+          <min>0.01</min>
+          <max>0.15</max>
+          <resolution>1.0</resolution>
+        </range>
+      </ray>
+    </sensor>
   </gazebo>
   <gazebo reference="cliff_sensor_right_link">
-    <sensor:ray name="cliff_sensor_right">
-      <alwaysActive>true</alwaysActive>
-      <rayCount>1</rayCount>
-      <rangeCount>1</rangeCount>
-      <resRange>0.1</resRange>
-      <minAngle>0</minAngle>
-      <maxAngle>0</maxAngle>
-      <minRange>0.01</minRange>
-      <maxRange>0.04</maxRange>
-      <displayRays>false</displayRays>
-    </sensor:ray>
+    <sensor type="ray" name="cliff_sensor_right">
+      <always_on>true</always_on>
+      <update_rate>50</update_rate>
+      <visualize>true</visualize>
+      <ray>
+        <scan>
+          <horizontal>
+            <samples>50</samples>
+            <resolution>1.0</resolution>
+            <min_angle>-0.0436</min_angle>  <!-- -2.5 degree -->
+            <max_angle>0.0436</max_angle> <!-- 2.5 degree -->
+          </horizontal>
+          <vertical>
+            <samples>50</samples>
+            <resolution>1.0</resolution>
+            <min_angle>-0.0436</min_angle>  <!-- -2.5 degree -->
+            <max_angle>0.0436</max_angle> <!-- 2.5 degree -->
+          </vertical>
+        </scan>
+        <range>
+          <min>0.01</min>
+          <max>0.15</max>
+          <resolution>1.0</resolution>
+        </range>
+      </ray>
+    </sensor>
   </gazebo>
   <gazebo reference="cliff_sensor_front_link">
-    <sensor:ray name="cliff_sensor_front">
-      <alwaysActive>true</alwaysActive>
-      <rayCount>1</rayCount>
-      <rangeCount>1</rangeCount>
-      <resRange>0.1</resRange>
-      <minAngle>0</minAngle>
-      <maxAngle>0</maxAngle>
-      <minRange>0.01</minRange>
-      <maxRange>0.04</maxRange>
-      <displayRays>false</displayRays>
-    </sensor:ray>
+    <sensor type="ray" name="cliff_sensor_front">
+      <always_on>true</always_on>
+      <update_rate>50</update_rate>
+      <visualize>true</visualize>
+      <ray>
+        <scan>
+          <horizontal>
+            <samples>50</samples>
+            <resolution>1.0</resolution>
+            <min_angle>-0.0436</min_angle>  <!-- -2.5 degree -->
+            <max_angle>0.0436</max_angle> <!-- 2.5 degree -->
+          </horizontal>
+          <vertical>
+            <samples>50</samples>
+            <resolution>1.0</resolution>
+            <min_angle>-0.0436</min_angle>  <!-- -2.5 degree -->
+            <max_angle>0.0436</max_angle> <!-- 2.5 degree -->
+          </vertical>
+        </scan>
+        <range>
+          <min>0.01</min>
+          <max>0.15</max>
+          <resolution>1.0</resolution>
+        </range>
+      </ray>
+    </sensor>
   </gazebo>
-</xacro:macro>
-<xacro:macro name="turtlebot_sim_imu">
   <gazebo>
-    <controller:gazebo_ros_imu name="imu_controller" plugin="libgazebo_ros_imu.so">
+    <plugin name="imu_controller" filename="libgazebo_ros_imu.so">
       <alwaysOn>true</alwaysOn>
-      <updateRate>30</updateRate>
+      <updateRate>50</updateRate>
       <bodyName>gyro_link</bodyName>
-      <topicName>imu/data</topicName>
+      <topicName>/mobile_base/sensors/imu_data</topicName>
       <gaussianNoise>${0.0017*0.0017}</gaussianNoise>
       <xyzOffsets>0 0 0</xyzOffsets>
       <rpyOffsets>0 0 0</rpyOffsets>
-      <interface:position name="gyro_link"/>
-    </controller:gazebo_ros_imu>
+    </plugin>
   </gazebo>
-</xacro:macro>
+  <gazebo>
+    <plugin name="kobuki_controller" filename="libgazebo_ros_kobuki.so">
+      <left_wheel_joint_name>wheel_left_joint</left_wheel_joint_name>
+      <right_wheel_joint_name>wheel_right_joint</right_wheel_joint_name>
+      <wheel_separation>.230</wheel_separation>
+      <wheel_diameter>0.070</wheel_diameter>
+      <torque>1.0</torque>
+      <velocity_command_timeout>0.6</velocity_command_timeout>
+      <cliff_sensor_left_name>cliff_sensor_left</cliff_sensor_left_name>
+      <cliff_sensor_front_name>cliff_sensor_front</cliff_sensor_front_name>
+      <cliff_sensor_right_name>cliff_sensor_right</cliff_sensor_right_name>
+      <cliff_detection_threshold>0.04</cliff_detection_threshold>
+      <bumper_name>bumpers</bumper_name>
+      <base_collision_model_link>base_link</base_collision_model_link>
+    </plugin>
+  </gazebo>
 </robot>

Commit message: Rebase from 'upstream'

File: kobuki_description/urdf/kobuki.urdf.xacro (robot description, xacro)
@@ -36,5 +36,5 @@
       <collision>
         <geometry>
-          <cylinder length="0.10938" radius="0.176"/>
+          <cylinder length="0.10938" radius="0.178"/>
         </geometry>
         <origin xyz="0.0 0 0.05949" rpy="0 0 0"/>

File: kobuki_description/urdf/kobuki_gazebo.urdf.xacro (robot description, xacro)
@@ -49,10 +49,12 @@
 	            <max_angle>0.0436</max_angle> <!-- 2.5 degree -->
 	          </horizontal>
-	          <vertical>
-	            <samples>50</samples>
-	            <resolution>1.0</resolution>
-	            <min_angle>-0.0436</min_angle>  <!-- -2.5 degree -->
-	            <max_angle>0.0436</max_angle> <!-- 2.5 degree -->
-	          </vertical>
+<!--            Can't use vertical rays until this bug is resolved: -->
+<!--            https://bitbucket.org/osrf/gazebo/issue/509/vertical-sensor-doesnt-works -->
+<!-- 	          <vertical> -->
+<!-- 	            <samples>50</samples> -->
+<!-- 	            <resolution>1.0</resolution> -->
+<!-- 	            <min_angle>-0.0436</min_angle>  -2.5 degree -->
+<!-- 	            <max_angle>0.0436</max_angle> 2.5 degree -->
+<!-- 	          </vertical> -->
 	        </scan>
 	        <range>
@@ -77,10 +79,12 @@
 	            <max_angle>0.0436</max_angle> <!-- 2.5 degree -->
 	          </horizontal>
-	          <vertical>
-	            <samples>50</samples>
-	            <resolution>1.0</resolution>
-	            <min_angle>-0.0436</min_angle>  <!-- -2.5 degree -->
-	            <max_angle>0.0436</max_angle> <!-- 2.5 degree -->
-	          </vertical>
+<!--            Can't use vertical rays until this bug is resolved: -->
+<!--            https://bitbucket.org/osrf/gazebo/issue/509/vertical-sensor-doesnt-works -->
+<!-- 	          <vertical> -->
+<!-- 	            <samples>50</samples> -->
+<!-- 	            <resolution>1.0</resolution> -->
+<!-- 	            <min_angle>-0.0436</min_angle>  -2.5 degree -->
+<!-- 	            <max_angle>0.0436</max_angle> 2.5 degree -->
+<!-- 	          </vertical> -->
 	        </scan>
 	        <range>
@@ -105,10 +109,12 @@
 	            <max_angle>0.0436</max_angle> <!-- 2.5 degree -->
 	          </horizontal>
-	          <vertical>
-	            <samples>50</samples>
-	            <resolution>1.0</resolution>
-	            <min_angle>-0.0436</min_angle>  <!-- -2.5 degree -->
-	            <max_angle>0.0436</max_angle> <!-- 2.5 degree -->
-	          </vertical>
+<!-- 	          Can't use vertical rays until this bug is resolved: -->
+<!--            https://bitbucket.org/osrf/gazebo/issue/509/vertical-sensor-doesnt-works -->
+<!-- 	          <vertical> -->
+<!-- 	            <samples>50</samples> -->
+<!-- 	            <resolution>1.0</resolution> -->
+<!-- 	            <min_angle>-0.0436</min_angle>  -2.5 degree -->
+<!-- 	            <max_angle>0.0436</max_angle> 2.5 degree -->
+<!-- 	          </vertical> -->
 	        </scan>
 	        <range>
